File: PCB/JediLightSwitch-V1.1.sch (EAGLE design)
At the start: 36 parts, among them U1 APDS-9960, U2 HTU21DSMD, U3 PHOTON_SMD, U4 AT42QT1010SOT23

Commit message: Removed V1.0 pdf's from this V1.1 branch.
Updated V1.1 pdf's for the V1.1.1 modification (moved 3v3 rail away from I2C pullups).
Other:
- note added: "1.1.1"
- note removed: "1.1"
Changed lines of the file:
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@@
 68nF sensitive without touch</text>
 <text x="178.562" y="-82.55" size="2.54" layer="97">Stephen Harrison</text>
-<text x="248.92" y="-86.36" size="2.54" layer="97">1.1</text>
+<text x="248.92" y="-86.36" size="2.54" layer="97">1.1.1</text>
 <text x="25.4" y="-91.44" size="1.6764" layer="97">Sparkfun Eagle Library and breakout boards for HTU21D, APDS-9960 &amp; AT42QT1010 used under CC. See Readme.md</text>
 <text x="27.94" y="-27.94" size="2.54" layer="97">Reverse mount LEDs.</text>
