File: V1.2/PCB/JediLightSwitch-V1.2.brd (EAGLE design)
At the start: 100 x 100 mm, 73 parts, among them U1 APDS-9960, U2 HTU21DSMD, U3 PHOTON_SMD, U4 AT42QT1010SOT23, U5 TEMT6000, U6 MCP73831, U7 MAX1704X

Commit message: Added part values
Parts:
- Q1: value (none) -> BSS138
Changed lines of the file:
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@@
 <attribute name="VALUE" x="19.812" y="33.5915" size="0.0254" layer="28" rot="MR0"/>
 </element>
-<element name="Q1" library="SparkFun-DiscreteSemi" package="SOT23-3" value="" x="26.3525" y="94.9325" rot="MR0">
+<element name="Q1" library="SparkFun-DiscreteSemi" package="SOT23-3" value="BSS138" x="26.3525" y="94.9325" rot="MR0">
 <attribute name="PROD_ID" value="TRAN-12988" x="26.3525" y="94.9325" size="0.8128" layer="28" font="vector" rot="MR0" display="off"/>
+<attribute name="FARNELL" value="9845330" x="26.3525" y="94.9325" size="1.778" layer="28" rot="MR0" display="off"/>
 </element>
 <element name="R18" library="rcl" package="R0805" value="10R" x="11.1125" y="92.075" smashed="yes" rot="MR270">
