File: V1.2/PCB/JediLightSwitch-V1.2.sch (EAGLE design)
At the start: 73 parts, among them Q1 MOSFET-NCHANNELAO3404A, U1 APDS-9960, U2 HTU21DSMD, U3 PHOTON_SMD, U4 AT42QT1010SOT23, U5 TEMT6000, U6 MCP73831, U7 MAX1704X

Commit message: Added part values
Parts:
- Q1: value MOSFET-NCHANNELAO3404A -> BSS138; FARNELL (none) -> 9845330
Changed lines of the file:
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@@
 <part name="GND25" library="SparkFun-Aesthetics" deviceset="DGND" device=""/>
 <part name="TP2" library="testpad" deviceset="TP" device="TP20R"/>
-<part name="Q1" library="SparkFun-DiscreteSemi" deviceset="MOSFET-NCHANNEL" device="AO3404A" value=""/>
+<part name="Q1" library="SparkFun-DiscreteSemi" deviceset="MOSFET-NCHANNEL" device="AO3404A" value="BSS138">
+<attribute name="FARNELL" value="9845330"/>
+</part>
 <part name="R18" library="rcl" deviceset="R-EU_" device="R0805" value="10R"/>
 <part name="R19" library="rcl" deviceset="R-EU_" device="R0805" value="10k"/>
@@
 <attribute name="NAME" x="274.32" y="-53.34" size="1.778" layer="95"/>
 <attribute name="VALUE" x="271.78" y="-55.88" size="1.778" layer="96"/>
+<attribute name="FARNELL" x="271.78" y="-48.26" size="1.778" layer="96" display="off"/>
 </instance>
 <instance part="R18" gate="G$1" x="254" y="-40.64" rot="R90"/>
